File: pcb/pcb.kicad_pcb (KiCad board)
At the start: 2 copper layers, 81 parts, among them J1 USB_B_Micro, J2 battery, J3 SD_Card, J4 swd, J5 speakers, SW1 RotaryEncoder, SW2 next, SW3 play, U1 TP4056, U2 LM358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

Commit message: pcb block wiev
Parts:
- removed C10, C8: 0.1, Capacitor_SMD:C_0402_1005Metric
- added C35: 0.1, Capacitor_SMD:C_0402_1005Metric, F.Cu at (120.0, 63.1)
- L1: footprint Inductor_SMD:L_0603_1608Metric -> Inductor_SMD:L_1206_3216Metric
- L2: moved to B.Cu
- U3: footprint Package_SO:SOIC-8-N7_3.9x4.9mm_P1.27mm -> Package_SO:SOP-8_3.9x4.9mm_P1.27mm
- moved J3 99.4 mm to (221.7, 67.7)
- moved R14 75.2 mm to (111.4, 61.6), turned to 180 degrees
- moved C13 73.2 mm to (114.0, 85.9)
- moved U7 71.6 mm to (152.5, 62.4), turned to 180 degrees
- moved U2 70.5 mm to (118.8, 58.8), turned to 90 degrees
- moved SW2 69.9 mm to (156.5, 89.9), turned to 180 degrees
- moved C31 68.6 mm to (109.6, 61.2), turned to 90 degrees
- moved R13 66.9 mm to (112.9, 53.0), turned to -90 degrees
- moved C21 63.4 mm to (118.8, 54.3)
- moved SW3 62.7 mm to (156.5, 82.3), turned to 180 degrees
- moved U6 60.2 mm to (112.4, 58.1), turned to 90 degrees
- moved C29 59.1 mm to (136.0, 86.7), turned to -90 degrees
- moved R8 59.1 mm to (116.5, 65.2), turned to 90 degrees
- moved C5 57.7 mm to (132.9, 75.0), turned to 180 degrees
- moved U4 55.5 mm to (127.7, 56.5)
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Connections:
- C2 pad 1: +4V -> +6V
- U1 pad 6: Net-(D1-Pad1) -> Net-(D1-Pad2)
- U1 pad 7: Net-(D1-Pad2) -> Net-(D1-Pad1)
- U4 pad 7: Net-(R6-Pad1) -> Net-(R7-Pad1)
- U4 pad 8: Net-(R7-Pad1) -> Net-(R6-Pad1)
- U7 pad 4: (no net) -> GND
- U7 pad 8: (no net) -> +6V
Routing:
- net GND: track 0.00 -> 83.2 mm, vias 0 -> 4
- net +6V: track 0.00 -> 52.3 mm, vias 0 -> 1
- net Net-(U2-Pad5): track 0.00 -> 23.7 mm, vias 0 -> 2
- net +4V: track 0.00 -> 19.6 mm
- net Net-(C1-Pad1): track 0.00 -> 17.3 mm
- net Net-(C34-Pad2): track 0.00 -> 10.6 mm
- net Net-(C33-Pad1): track 0.00 -> 10.5 mm
- net Net-(R6-Pad1): track 0.00 -> 9.56 mm
- net Net-(D2-Pad2): track 0.00 -> 9.43 mm
- net Net-(R7-Pad1): track 0.00 -> 9.18 mm
- net /MIC: track 0.00 -> 8.58 mm
- net Net-(C20-Pad1): track 0.00 -> 6.99 mm
- net Net-(C23-Pad1): track 0.00 -> 6.87 mm
- net Net-(C22-Pad1): track 0.00 -> 6.19 mm
- net Net-(C14-Pad1): track 0.00 -> 5.73 mm, vias 0 -> 1
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
Commit message: 4.5x4 pcb
Parts:
- C31, C32: footprint Capacitor_Tantalum_SMD:CP_EIA-1608-08_AVX-J -> Capacitor_Tantalum_SMD:CP_EIA-3216-10_Kemet-I
- J4: footprint Connector_PinHeader_1.00mm:PinHeader_1x04_P1.00mm_Vertical_SMD_Pin1Left -> local:swd
- L2: moved to F.Cu
- moved J3 97.2 mm to (124.5, 67.1)
- moved R18 22.6 mm to (135.0, 60.2), turned to 90 degrees
- moved C33 21.4 mm to (136.0, 60.2), turned to -90 degrees
- moved R16 19.8 mm to (137.5, 60.2), turned to 90 degrees
- moved R17 18.5 mm to (133.5, 57.1), turned to 90 degrees
- moved R19 18.0 mm to (139.3, 59.7)
- moved U7 17.2 mm to (136.8, 55.4), turned to 90 degrees
- moved C34 15.2 mm to (142.1, 59.6), turned to 0 degrees
- moved SW1 14.1 mm to (143.6, 65.5)
- moved R20 11.7 mm to (140.1, 53.1), turned to 90 degrees
- moved J4 9.90 mm to (140.1, 63.9), turned to -90 degrees
- moved MK1 9.83 mm to (143.6, 55.6), turned to 180 degrees
- moved SW3 9.17 mm to (149.4, 76.4)
- moved SW2 9.16 mm to (149.4, 84.1)
- moved C14 8.70 mm to (131.2, 58.0), turned to -90 degrees
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Connections:
- J3 pad 2: Net-(J3-Pad2) -> Net-(U5-Pad16)
- J3 pad 5: Net-(J3-Pad5) -> Net-(U5-Pad20)
- U4 pad 7: Net-(R7-Pad1) -> Net-(R6-Pad1)
- U4 pad 8: Net-(R6-Pad1) -> Net-(R7-Pad1)
- U5 pad 15: Net-(J3-Pad7) -> Net-(J3-Pad1)
- U5 pad 16: Net-(J3-Pad5) -> Net-(U5-Pad16)
- U5 pad 20: Net-(J3-Pad2) -> Net-(U5-Pad20)
- U5 pad 21: Net-(J3-Pad1) -> Net-(J3-Pad7)
- U5 pad 24: /ADC_SCK -> /ADC_LRCLK
- U5 pad 25: /ADC_BCK -> /ADC_DATA
- U5 pad 26: /ADC_DATA -> /ADC_BCK
- U5 pad 27: /ADC_LRCLK -> /ADC_SCK
- U5 pad 4: unconnected-(U5-Pad4) -> GND
- U5 pad 5: unconnected-(U5-Pad5) -> GND
Routing:
- net GND: track 83.2 -> 236.7 mm
- net +4V: track 19.6 -> 123.8 mm, vias 0 -> 2
- net Net-(J3-Pad1): track 0.00 -> 65.5 mm, vias 0 -> 1
- net Net-(U5-Pad16): track 0.00 -> 61.7 mm, vias 0 -> 1
- net +6V: track 52.3 -> 113.7 mm, vias 1 -> 4
- net Net-(U5-Pad20): track 0.00 -> 50.9 mm, vias 0 -> 1
- net /PA_SDN: track 0.00 -> 43.1 mm
- net Net-(J3-Pad7): track 0.00 -> 42.2 mm, vias 0 -> 1
- net +VSW: track 0.00 -> 35.0 mm, vias 0 -> 3
- net Net-(SW1-PadB): track 0.00 -> 29.9 mm
- net Net-(SW1-PadC): track 0.00 -> 25.6 mm
- net Net-(SW1-PadA): track 0.00 -> 19.7 mm
- net Net-(SW3-Pad2): track 0.00 -> 19.5 mm
- net /ADC_SCK: track 0.00 -> 18.6 mm
- net Net-(SW2-Pad2): track 0.00 -> 17.3 mm
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- added copper zone on F.Cu, net GND
